Commit message: URDF practice

File: robot_modeling_ws/src/robot_description_pkg/urdf/test_3.urdf (robot description, URDF)
Before this commit: robot test_3, 4 links, 3 joints
Joints:
- joint base_vertical_move: axis (none) -> 0 1 0; limit (none) -> lower=-1.57 upper=1.57 effort=30 velocity=1.0; origin xyz=0 0 0.05 -> xyz=0 0 0.1; type fixed -> revolute
- joint vertical_horizontal: origin xyz=0 0 0.1 -> xyz=0 0 0.2
