Commit message: Add gripper and colours to differentiate links

File: robot_modeling_ws/src/robot_description_pkg/urdf/panda_based_arm.urdf (robot description, URDF)
Before this commit: robot panda_based_arm, 16 links, 15 joints
Links:
- added link gripper_link_1; visual box size=0.025 0.025 0.05
- added link gripper_link_2; visual box size=0.025 0.025 0.05
Joints:
- added joint hand-gripper_link_1: type prismatic, parent hand, child gripper_link_1, origin xyz=0.0375 0 0.05, axis 1 0 0, limit lower=0 upper=-0.025 effort=100 velocity=1.0
- added joint hand-gripper_link_2: type prismatic, parent hand, child gripper_link_2, origin xyz=-0.0375 0 0.05, axis 1 0 0, limit lower=0 upper=0.025 effort=100 velocity=1.0

File: robot_modeling_ws/src/robot_description_pkg/urdf/panda_based_arm.xacro (robot description, xacro)
@@ -1,4 +1,10 @@
 <?xml version="1.0"?>
 <robot xmlns:xacro="http://www.ros.org/wiki/xacro" name="panda_based_arm">
+  <material name="Black">
+    <color rgba="0 0 0 1"/>
+  </material>
+  <material name="White">
+    <color rgba="1 1 1 1"/>
+  </material>
   <xacro:property name="link_1_length" value="0.1"/>
   <xacro:property name="link_2_length" value="0.1"/>
@@ -15,5 +21,8 @@
   <xacro:property name="link_13_length" value="0.05"/>
   <xacro:property name="hand_height" value="0.05"/>
-  <xacro:property name="hand_size" value="0.1 0.025 ${hand_height}"/>
+  <xacro:property name="hand_length" value="0.1"/>
+  <xacro:property name="gripper_length" value="0.05"/>
+  <xacro:property name="stationary_link_color" value="Black"/>
+  <xacro:property name="rotating_link_colour" value="White"/>
   <xacro:macro name="cylinder_link" params="name length xyz rpy">
     <link name="${name}">
@@ -23,4 +32,5 @@
         </geometry>
         <origin xyz="${xyz}" rpy="${rpy}"/>
+        <material name="${rotating_link_colour}"/>
       </visual>
     </link>
@@ -33,4 +43,16 @@
         </geometry>
         <origin xyz="${xyz}" rpy="${rpy}"/>
+        <material name="${stationary_link_color}"/>
+      </visual>
+    </link>
+  </xacro:macro>
+  <xacro:macro name="gripper_link" params="name xyz rpy">
+    <link name="${name}">
+      <visual>
+        <geometry>
+          <box size="0.025 0.025 ${gripper_length}"/>
+        </geometry>
+        <origin xyz="${xyz}" rpy="${rpy}"/>
+        <material name="${rotating_link_colour}"/>
       </visual>
     </link>
@@ -50,4 +72,13 @@
       <child link="${child}"/>
       <origin xyz="${xyz}"/>
+    </joint>
+  </xacro:macro>
+  <xacro:macro name="gripper_joint" params="name parent child xyz axis lower upper">
+    <joint name="${name}" type="prismatic">
+      <parent link="${parent}"/>
+      <child link="${child}"/>
+      <origin xyz="${xyz}"/>
+      <axis xyz="${axis}"/>
+      <limit effort="100" velocity="1.0" lower="${lower}" upper="${upper}"/>
     </joint>
   </xacro:macro>
@@ -206,8 +237,28 @@
       <visual>
         <geometry>
-          <box size="${hand_size}"/>
+          <box size="${hand_length} 0.025 ${hand_height}"/>
         </geometry>
         <origin xyz="0 0 ${hand_height/2}"/>
       </visual>
     </link>
+    <xacro:gripper_joint name="hand-gripper_link_1"
+      parent="hand"
+      child="gripper_link_1"
+      xyz="${hand_length/2-0.0125} 0 ${hand_height}"
+      axis="1 0 0"
+      lower="0"
+      upper="${0.025-hand_length/2}"/>
+    <xacro:gripper_link name="gripper_link_1"
+      xyz="0 0 ${gripper_length/2}"
+      rpy="0 0 0"/>
+    <xacro:gripper_joint name="hand-gripper_link_2"
+      parent="hand"
+      child="gripper_link_2"
+      xyz="${0.0125-hand_length/2} 0 ${hand_height}"
+      axis="1 0 0"
+      lower="0"
+      upper="${hand_length/2-0.025}"/>
+    <xacro:gripper_link name="gripper_link_2"
+      xyz="0 0 ${gripper_length/2}"
+      rpy="0 0 0"/>
 </robot>
