Commit message: Calculate and add inertia matrix to the links

File: robot_modeling_ws/src/robot_description_pkg/urdf/mesh_arm.urdf (robot description, URDF)
Before this commit: robot seven_dof_arm_using_mesh, 8 links, 7 joints
Links:
- link link_1: mass None -> 0.5
- link link_2: mass None -> 0.5
- link link_3: mass None -> 0.5
- link link_4: mass None -> 0.5
- link link_5: mass None -> 0.5
- link link_6: mass None -> 0.5
- link link_7: mass None -> 0.5

File: robot_modeling_ws/src/robot_description_pkg/urdf/mesh_arm.xacro (robot description, xacro)
@@ -15,11 +15,5 @@
   <xacro:property name="link_6_mesh" value="package://robot_description_pkg/meshes/link_4.stl"/>
   <xacro:property name="link_7_mesh" value="package://robot_description_pkg/meshes/link_5.stl"/>
-  <xacro:macro name="inertial_matrix" params="mass ixx ixy ixz iyy iyz izz">
-    <inertial>
-      <mass value="${mass}"/>
-      <inertia ixx="${ixx}" ixy="${ixy}" ixz="${ixz}" iyy="${iyy}" iyz="${iyz}" izz="${izz}"/>
-    </inertial>
-  </xacro:macro>
-  <xacro:macro name="make_link" params="name mesh xyz rpy color">
+  <xacro:macro name="make_link" params="name mesh xyz rpy color mass ixx ixy ixz iyy iyz izz">
     <link name="${name}">
       <visual>
@@ -36,4 +30,8 @@
         <origin xyz="${xyz}" rpy="${rpy}"/>
       </collision>
+      <inertial>
+        <mass value="${mass}"/>
+        <inertia ixx="${ixx}" ixy="${ixy}" ixz="${ixz}" iyy="${iyy}" iyz="${iyz}" izz="${izz}"/>
+      </inertial>
     </link>
   </xacro:macro>
@@ -54,9 +52,19 @@
     </joint>
   </xacro:macro>
-  <xacro:make_link name="base_link"
-    mesh="${base_link_mesh}"
-    xyz="0 0 0"
-    rpy="0 0 0"
-    color="White"/>
+  <link name="base_link">
+    <visual>
+      <geometry>
+        <mesh filename="${base_link_mesh}" scale="0.001 0.001 0.001"/>
+      </geometry>
+      <origin xyz="0 0 0" rpy="0 0 0"/>
+      <material name="White"/>
+    </visual>
+    <collision>
+      <geometry>
+        <mesh filename="${base_link_mesh}" scale="0.0011 0.0011 0.0011"/>
+      </geometry>
+      <origin xyz="0 0 0" rpy="0 0 0"/>
+    </collision>
+  </link>
   <xacro:join_links name="base_link-link_1"
     parent="base_link"
@@ -70,5 +78,9 @@
     xyz="0 0 0"
     rpy="0 0 0"
-    color="Black"/>
+    color="Black"
+    mass="0.5"
+    ixx="160347952.000000" ixy="0.073988" ixz="15663199.000000"
+    iyy="149014144.000000" iyz="0.506316"
+    izz="44131488.000000"/>
   <xacro:join_links name="link_1-link_2"
     parent="link_1"
@@ -82,5 +94,9 @@
     xyz="0 0 0"
     rpy="0 0 0"
-    color="White"/>
+    color="White"
+    mass="0.5"
+    ixx="320315008.000000" ixy="0.025285" ixz="1.992257"
+    iyy="295672384.000000" iyz="0.107130"
+    izz="42775932.000000"/>
   <xacro:join_links name="link_2-link_3"
     parent="link_2"
@@ -94,5 +110,9 @@
     xyz="0 0 0"
     rpy="0 0 0"
-    color="Black"/>
+    color="Black"
+    mass="0.5"
+    ixx="93527256.000000" ixy="0.003871" ixz="12514371.000000"
+    iyy="87003976.000000" iyz="0.035148"
+    izz="40058448.000000"/>
   <xacro:join_links name="link_3-link_4"
     parent="link_3"
@@ -106,5 +126,9 @@
     xyz="0 0 0"
     rpy="0 0 0"
-    color="White"/>
+    color="White"
+    mass="0.5"
+    ixx="93527256.000000" ixy="0.003871" ixz="12514371.000000"
+    iyy="87003976.000000" iyz="0.035148"
+    izz="40058448.000000"/>
   <xacro:join_links name="link_4-link_5"
     parent="link_4"
@@ -118,5 +142,9 @@
     xyz="0 0 0"
     rpy="0 0 3.14"
-    color="Black"/>
+    color="Black"
+    mass="0.5"
+    ixx="93527256.000000" ixy="0.003871" ixz="12514371.000000"
+    iyy="87003976.000000" iyz="0.035148"
+    izz="40058448.000000"/>
   <xacro:join_links name="link_5-link_6"
     parent="link_5"
@@ -130,5 +158,9 @@
     xyz="0 0 0"
     rpy="0 0 3.14"
-    color="White"/>
+    color="White"
+    mass="0.5"
+    ixx="93527256.000000" ixy="0.003871" ixz="12514371.000000"
+    iyy="87003976.000000" iyz="0.035148"
+    izz="40058448.000000"/>
   <xacro:join_links name="link_6-link_7"
     parent="link_6"
@@ -142,4 +174,8 @@
     xyz="0 0 0"
     rpy="0 0 0"
-    color="Black"/>
+    color="Black"
+    mass="0.5"
+    ixx="130744760.000000" ixy="0.001162" ixz="20542782.000000"
+    iyy="127046656.000000" iyz="0.004876"
+    izz="49867952.000000"/>
 </robot>

Commit message: Add hand and finger to the arm

File: robot_modeling_ws/src/robot_description_pkg/urdf/mesh_arm.urdf (robot description, URDF)
Before this commit: robot seven_dof_arm_using_mesh, 8 links, 7 joints
Links:
- added link finger_1, mass 0.25; collision mesh filename=package://robot_description_pkg/meshes/finger.stl scale=0.0011 0.0011 0.0011; visual mesh filename=package://robot_description_pkg/meshes/finger.stl scale=0.001 0.001 0.001
- added link finger_2, mass 0.25; collision mesh filename=package://robot_description_pkg/meshes/finger.stl scale=0.0011 0.0011 0.0011; visual mesh filename=package://robot_description_pkg/meshes/finger.stl scale=0.001 0.001 0.001
- added link hand, mass 0.5; collision mesh filename=package://robot_description_pkg/meshes/hand.stl scale=0.0011 0.0011 0.0011; visual mesh filename=package://robot_description_pkg/meshes/hand.stl scale=0.001 0.001 0.001
Joints:
- added joint hand-finger: type prismatic, parent hand, child finger_1, origin xyz=0.03 0 0.04, limit lower=0 upper=-0.03 effort=100 velocity=1.0
- added joint hand-finger_2: type prismatic, parent hand, child finger_2, origin xyz=-0.03 0 0.04, limit lower=0 upper=0.03 effort=100 velocity=1.0, mimic joint=hand-finger multiplier=-1
- added joint link_7-hand: type fixed, parent link_7, child hand, origin xyz=0 0 0.085

File: robot_modeling_ws/src/robot_description_pkg/urdf/mesh_arm.xacro (robot description, xacro)
@@ -17,4 +17,6 @@
   <xacro:property name="link_6_mesh" value="package://robot_description_pkg/meshes/link_4.stl"/>
   <xacro:property name="link_7_mesh" value="package://robot_description_pkg/meshes/link_5.stl"/>
+  <xacro:property name="hand_mesh" value="package://robot_description_pkg/meshes/hand.stl"/>
+  <xacro:property name="finger_mesh" value="package://robot_description_pkg/meshes/finger.stl"/>
   <xacro:macro name="make_link" params="name mesh xyz rpy color mass ixx ixy ixz iyy iyz izz">
     <link name="${name}">
@@ -181,3 +183,47 @@
     iyy="127046656.000000" iyz="0.004876"
     izz="49867952.000000"/>
+  <xacro:fix_links name="link_7-hand"
+    parent="link_7"
+    child="hand"
+    xyz="0 0 0.085"/>
+  <xacro:make_link name="hand"
+    mesh="${hand_mesh}"
+    xyz="0 0 0"
+    rpy="0 0 0"
+    color="White"
+    mass="0.5"
+    ixx="13535881.000000" ixy="0.005851" ixz="0.209502"
+    iyy="48692132.000000" iyz="0.001552"
+    izz="42968752.000000"/>
+  <joint name="hand-finger" type="prismatic">
+    <parent link="hand"/>
+    <child link="finger_1"/>
+    <origin xyz="0.03 0 0.04"/>
+    <limit effort="100" velocity="1.0" lower="0" upper="-0.03"/>
+  </joint>
+  <xacro:make_link name="finger_1"
+    mesh="${finger_mesh}"
+    xyz="0 0 0"
+    rpy="0 0 0"
+    color="Black"
+    mass="0.25"
+    ixx="1640625.000000" ixy="0.000262" ixz="416666.656250"
+    iyy="1453125.500000" iyz="0.000365"
+    izz="593749.937500"/>
+  <joint name="hand-finger_2" type="prismatic">
+    <parent link="hand"/>
+    <child link="finger_2"/>
+    <origin xyz="-0.03 0 0.04"/>
+    <limit effort="100" velocity="1.0" lower="0" upper="0.03"/>
+    <mimic joint="hand-finger" multiplier="-1"/>
+  </joint>
+  <xacro:make_link name="finger_2"
+    mesh="${finger_mesh}"
+    xyz="0 0 0"
+    rpy="0 0 3.14"
+    color="Black"
+    mass="0.25"
+    ixx="1640625.000000" ixy="0.000262" ixz="416666.656250"
+    iyy="1453125.500000" iyz="0.000365"
+    izz="593749.937500"/>
 </robot>

Commit message: Set end effector and disable unwanted collisions

File: robot_modeling_ws/src/robot_description_pkg/urdf/mesh_arm.urdf (robot description, URDF)
Before this commit: robot seven_dof_arm_using_mesh, 11 links, 10 joints
Joints:
- joint link_1-link_2: limit lower=-1.57 upper=1.57 effort=300 velocity=0.1 -> lower=-2.3 upper=2.3 effort=300 velocity=0.1
- joint link_2-link_3: limit lower=-1.57 upper=1.57 effort=300 velocity=0.1 -> lower=-1.8 upper=1.8 effort=300 velocity=0.1
- joint link_3-link_4: limit lower=-1.57 upper=1.57 effort=300 velocity=0.1 -> lower=-3.14 upper=3.14 effort=300 velocity=0.1
- joint link_4-link_5: limit lower=-1.57 upper=1.57 effort=300 velocity=0.1 -> lower=-1.8 upper=1.8 effort=300 velocity=0.1
- joint link_5-link_6: limit lower=-1.57 upper=1.57 effort=300 velocity=0.1 -> lower=-3.14 upper=3.14 effort=300 velocity=0.1
- joint link_6-link_7: limit lower=-1.57 upper=1.57 effort=300 velocity=0.1 -> lower=-1.8 upper=1.8 effort=300 velocity=0.1

File: robot_modeling_ws/src/robot_description_pkg/urdf/mesh_arm.xacro (robot description, xacro)
@@ -9,4 +9,9 @@
   <xacro:include filename="$(find robot_description_pkg)/urdf/mesh_arm_grouping.xacro"/>
   <xacro:group_arm/>
+  <xacro:group_hand/>
+  <xacro:disable_unwanted_arm_collisions/>
+  <xacro:disable_unwanted_hand_collisions/>
+  <xacro:disable_unwanted_arm_hand_collisions/>
+  <end_effector name="hand" parent_link="link_7" group="hand_group" parent_group="arm_group"/>
   <xacro:property name="base_link_mesh" value="package://robot_description_pkg/meshes/base_link.stl"/>
   <xacro:property name="link_1_mesh" value="package://robot_description_pkg/meshes/link_1.stl"/>
@@ -92,6 +97,6 @@
     xyz="0 0 0.08"
     axis="1 0 0"
-    lower="-1.57"
-    upper="1.57"/>
+    lower="-2.3"
+    upper="2.3"/>
   <xacro:make_link name="link_2"
     mesh="${link_2_mesh}"
@@ -108,6 +113,6 @@
     xyz="0 0 0.1"
     axis="1 0 0"
-    lower="-1.57"
-    upper="1.57"/>
+    lower="-1.8"
+    upper="1.8"/>
   <xacro:make_link name="link_3"
     mesh="${link_3_mesh}"
@@ -124,6 +129,6 @@
     xyz="0 0 0.06"
     axis="0 0 1"
-    lower="-1.57"
-    upper="1.57"/>
+    lower="-3.14"
+    upper="3.14"/>
   <xacro:make_link name="link_4"
     mesh="${link_4_mesh}"
@@ -140,6 +145,6 @@
     xyz="0 0 0.06"
     axis="1 0 0"
-    lower="-1.57"
-    upper="1.57"/>
+    lower="-1.8"
+    upper="1.8"/>
   <xacro:make_link name="link_5"
     mesh="${link_5_mesh}"
@@ -156,6 +161,6 @@
     xyz="0 0 0.06"
     axis="0 0 1"
-    lower="-1.57"
-    upper="1.57"/>
+    lower="-3.14"
+    upper="3.14"/>
   <xacro:make_link name="link_6"
     mesh="${link_6_mesh}"
@@ -172,6 +177,6 @@
     xyz="0 0 0.06"
     axis="1 0 0"
-    lower="-1.57"
-    upper="1.57"/>
+    lower="-1.8"
+    upper="1.8"/>
   <xacro:make_link name="link_7"
     mesh="${link_7_mesh}"

File: robot_modeling_ws/src/robot_description_pkg/urdf/mesh_arm_grouping.xacro (robot description, xacro)
@@ -2,7 +2,61 @@
 <robot name="seven_dof_arm_using_mesh" xmlns:xacro="http://www.ros.org/wiki/xacro" >
   <xacro:macro name="group_arm">
-    <group name="mesh_arm">
+    <group name="arm_group">
       <chain base_link="base_link" tip_link="link_7"/>
     </group>
   </xacro:macro>
+  <xacro:macro name="group_hand">
+    <group name="hand_group">
+      <link name="hand"/>
+      <link name="finger_1"/>
+      <link name="finger_2"/>
+      <joint name="hand-finger"/>
+      <passive_joint name="hand-finger_2"/>
+    </group>
+  </xacro:macro>
+  <xacro:macro name="disable_unwanted_arm_collisions">
+    <disable_collision link1="base_link" link2="link_1" reason="Adjacent"/>
+    <disable_collision link1="link_1" link2="link_2" reason="Adjacent"/>
+    <disable_collision link1="link_2" link2="link_3" reason="Adjacent"/>
+    <disable_collision link1="link_3" link2="link_4" reason="Adjacent"/>
+    <disable_collision link1="link_4" link2="link_5" reason="Adjacent"/>
+    <disable_collision link1="link_5" link2="link_6" reason="Adjacent"/>
+    <disable_collision link1="link_6" link2="link_7" reason="Adjacent"/>
+    <disable_collision link1="base_link" link2="link_2" reason="Never"/>
+    <disable_collision link1="base_link" link2="link_3" reason="Never"/>
+    <disable_collision link1="link_1" link2="link_3" reason="Never"/>
+    <disable_collision link1="link_1" link2="link_4" reason="Never"/>
+    <disable_collision link1="link_1" link2="link_5" reason="Never"/>
+    <disable_collision link1="link_2" link2="link_4" reason="Never"/>
+    <disable_collision link1="link_2" link2="link_5" reason="Never"/>
+    <disable_collision link1="link_2" link2="link_6" reason="Never"/>
+    <disable_collision link1="link_3" link2="link_5" reason="Never"/>
+    <disable_collision link1="link_3" link2="link_6" reason="Never"/>
+    <disable_collision link1="link_3" link2="link_7" reason="Never"/>
+    <disable_collision link1="link_4" link2="link_6" reason="Never"/>
+    <disable_collision link1="link_4" link2="link_7" reason="Never"/>
+    <disable_collision link1="link_5" link2="link_7" reason="Never"/>
+  </xacro:macro>
+  <xacro:macro name="disable_unwanted_hand_collisions">
+    <disable_collision link1="hand" link2="finger_1" reason="Adjacent"/>
+    <disable_collision link1="hand" link2="finger_2" reason="Adjacent"/>
+    <disable_collision link1="finger_1" link2="finger_2" reason="Fingers"/>
+  </xacro:macro>
+  <xacro:macro name="disable_unwanted_arm_hand_collisions">
+    <disable_collision link1="hand" link2="link_7" reason="Adjacent"/>
+    <disable_collision link1="hand" link2="link_6" reason="Never"/>
+    <disable_collision link1="hand" link2="link_5" reason="Never"/>
+    <disable_collision link1="hand" link2="link_4" reason="Never"/>
+    <disable_collision link1="hand" link2="link_3" reason="Never"/>
+    <disable_collision link1="finger_1" link2="link_7" reason="Never"/>
+    <disable_collision link1="finger_1" link2="link_6" reason="Never"/>
+    <disable_collision link1="finger_1" link2="link_5" reason="Never"/>
+    <disable_collision link1="finger_1" link2="link_4" reason="Never"/>
+    <disable_collision link1="finger_1" link2="link_3" reason="Never"/>
+    <disable_collision link1="finger_2" link2="link_7" reason="Never"/>
+    <disable_collision link1="finger_2" link2="link_6" reason="Never"/>
+    <disable_collision link1="finger_2" link2="link_5" reason="Never"/>
+    <disable_collision link1="finger_2" link2="link_4" reason="Never"/>
+    <disable_collision link1="finger_2" link2="link_3" reason="Never"/>
+  </xacro:macro>
 </robot>

Commit message: Modify xacro to run on moveit setup assistant

File: robot_modeling_ws/src/robot_description_pkg/urdf/mesh_arm.urdf (robot description, URDF)
Before this commit: robot seven_dof_arm_using_mesh, 11 links, 10 joints
Links:
- link finger_1: mass 0.25 -> 0.01
- link finger_2: mass 0.25 -> 0.01
- link hand: mass 0.5 -> 0.075
- link link_1: mass 0.5 -> 0.075
- link link_2: mass 0.5 -> 0.075
- link link_3: mass 0.5 -> 0.075
- link link_4: mass 0.5 -> 0.075
- link link_5: mass 0.5 -> 0.075
- link link_6: mass 0.5 -> 0.075
- link link_7: mass 0.5 -> 0.075
Joints:
- removed joint base_link-link_1
- removed joint hand-finger
- removed joint hand-finger_2
- removed joint link_1-link_2
- removed joint link_2-link_3
- removed joint link_3-link_4
- removed joint link_4-link_5
- removed joint link_5-link_6
- removed joint link_6-link_7
- removed joint link_7-hand
- added joint base_link_link_1: type revolute, parent base_link, child link_1, origin xyz=0 0 0.06, axis 0 0 1, limit lower=-3.14 upper=3.14 effort=300 velocity=0.1
- added joint hand_finger_1: type prismatic, parent hand, child finger_1, origin xyz=0.03 0 0.04, limit lower=0 upper=-0.03 effort=100 velocity=1.0, mimic joint=hand_finger_2 multiplier=-1
- added joint hand_finger_2: type prismatic, parent hand, child finger_2, origin xyz=-0.03 0 0.04, limit lower=0 upper=0.03 effort=100 velocity=1.0
- added joint link_1_link_2: type revolute, parent link_1, child link_2, origin xyz=0 0 0.08, axis 1 0 0, limit lower=-2.3 upper=2.3 effort=300 velocity=0.1
- added joint link_2_link_3: type revolute, parent link_2, child link_3, origin xyz=0 0 0.1, axis 1 0 0, limit lower=-1.8 upper=1.8 effort=300 velocity=0.1
- added joint link_3_link_4: type revolute, parent link_3, child link_4, origin xyz=0 0 0.06, axis 0 0 1, limit lower=-3.14 upper=3.14 effort=300 velocity=0.1
- added joint link_4_link_5: type revolute, parent link_4, child link_5, origin xyz=0 0 0.06, axis 1 0 0, limit lower=-1.8 upper=1.8 effort=300 velocity=0.1
- added joint link_5_link_6: type revolute, parent link_5, child link_6, origin xyz=0 0 0.06, axis 0 0 1, limit lower=-3.14 upper=3.14 effort=300 velocity=0.1
- added joint link_6_link_7: type revolute, parent link_6, child link_7, origin xyz=0 0 0.06, axis 1 0 0, limit lower=-1.8 upper=1.8 effort=300 velocity=0.1
- added joint link_7_hand: type fixed, parent link_7, child hand, origin xyz=0 0 0.085

File: robot_modeling_ws/src/robot_description_pkg/urdf/mesh_arm.xacro (robot description, xacro)
@@ -1,4 +1,4 @@
 <?xml version="1.0"?>
-<robot name="seven_dof_arm_using_mesh" xmlns:xacro="http://www.ros.org/wiki/xacro" >
+<robot name="penguin" xmlns:xacro="http://www.ros.org/wiki/xacro" >
   <material name="Black">
     <color rgba="0.5 0.5 0.5 1"/>
@@ -7,11 +7,4 @@
     <color rgba="1 1 1 1"/>
   </material>
-  <xacro:include filename="$(find robot_description_pkg)/urdf/mesh_arm_grouping.xacro"/>
-  <xacro:group_arm/>
-  <xacro:group_hand/>
-  <xacro:disable_unwanted_arm_collisions/>
-  <xacro:disable_unwanted_hand_collisions/>
-  <xacro:disable_unwanted_arm_hand_collisions/>
-  <end_effector name="hand" parent_link="link_7" group="hand_group" parent_group="arm_group"/>
   <xacro:property name="base_link_mesh" value="package://robot_description_pkg/meshes/base_link.stl"/>
   <xacro:property name="link_1_mesh" value="package://robot_description_pkg/meshes/link_1.stl"/>
@@ -76,5 +69,5 @@
     </collision>
   </link>
-  <xacro:join_links name="base_link-link_1"
+  <xacro:join_links name="base_link_link_1"
     parent="base_link"
     child="link_1"
@@ -88,9 +81,9 @@
     rpy="0 0 0"
     color="Black"
-    mass="0.5"
+    mass="0.075"
     ixx="160347952.000000" ixy="0.073988" ixz="15663199.000000"
     iyy="149014144.000000" iyz="0.506316"
     izz="44131488.000000"/>
-  <xacro:join_links name="link_1-link_2"
+  <xacro:join_links name="link_1_link_2"
     parent="link_1"
     child="link_2"
@@ -104,9 +97,9 @@
     rpy="0 0 0"
     color="White"
-    mass="0.5"
+    mass="0.075"
     ixx="320315008.000000" ixy="0.025285" ixz="1.992257"
     iyy="295672384.000000" iyz="0.107130"
     izz="42775932.000000"/>
-  <xacro:join_links name="link_2-link_3"
+  <xacro:join_links name="link_2_link_3"
     parent="link_2"
     child="link_3"
@@ -120,9 +113,9 @@
     rpy="0 0 0"
     color="Black"
-    mass="0.5"
-    ixx="93527256.000000" ixy="0.003871" ixz="12514371.000000"
-    iyy="87003976.000000" iyz="0.035148"
-    izz="40058448.000000"/>
-  <xacro:join_links name="link_3-link_4"
+    mass="0.075"
+    ixx="93527256.000000" ixy="0.003871" ixz="12514371.000000"
+    iyy="87003976.000000" iyz="0.035148"
+    izz="40058448.000000"/>
+  <xacro:join_links name="link_3_link_4"
     parent="link_3"
     child="link_4"
@@ -136,9 +129,9 @@
     rpy="0 0 0"
     color="White"
-    mass="0.5"
-    ixx="93527256.000000" ixy="0.003871" ixz="12514371.000000"
-    iyy="87003976.000000" iyz="0.035148"
-    izz="40058448.000000"/>
-  <xacro:join_links name="link_4-link_5"
+    mass="0.075"
+    ixx="93527256.000000" ixy="0.003871" ixz="12514371.000000"
+    iyy="87003976.000000" iyz="0.035148"
+    izz="40058448.000000"/>
+  <xacro:join_links name="link_4_link_5"
     parent="link_4"
     child="link_5"
@@ -152,9 +145,9 @@
     rpy="0 0 3.14"
     color="Black"
-    mass="0.5"
-    ixx="93527256.000000" ixy="0.003871" ixz="12514371.000000"
-    iyy="87003976.000000" iyz="0.035148"
-    izz="40058448.000000"/>
-  <xacro:join_links name="link_5-link_6"
+    mass="0.075"
+    ixx="93527256.000000" ixy="0.003871" ixz="12514371.000000"
+    iyy="87003976.000000" iyz="0.035148"
+    izz="40058448.000000"/>
+  <xacro:join_links name="link_5_link_6"
     parent="link_5"
     child="link_6"
@@ -168,9 +161,9 @@
     rpy="0 0 3.14"
     color="White"
-    mass="0.5"
-    ixx="93527256.000000" ixy="0.003871" ixz="12514371.000000"
-    iyy="87003976.000000" iyz="0.035148"
-    izz="40058448.000000"/>
-  <xacro:join_links name="link_6-link_7"
+    mass="0.075"
+    ixx="93527256.000000" ixy="0.003871" ixz="12514371.000000"
+    iyy="87003976.000000" iyz="0.035148"
+    izz="40058448.000000"/>
+  <xacro:join_links name="link_6_link_7"
     parent="link_6"
     child="link_7"
@@ -184,9 +177,9 @@
     rpy="0 0 0"
     color="Black"
-    mass="0.5"
+    mass="0.075"
     ixx="130744760.000000" ixy="0.001162" ixz="20542782.000000"
     iyy="127046656.000000" iyz="0.004876"
     izz="49867952.000000"/>
-  <xacro:fix_links name="link_7-hand"
+  <xacro:fix_links name="link_7_hand"
     parent="link_7"
     child="hand"
@@ -197,13 +190,14 @@
     rpy="0 0 0"
     color="White"
-    mass="0.5"
+    mass="0.075"
     ixx="13535881.000000" ixy="0.005851" ixz="0.209502"
     iyy="48692132.000000" iyz="0.001552"
     izz="42968752.000000"/>
-  <joint name="hand-finger" type="prismatic">
+  <joint name="hand_finger_1" type="prismatic">
     <parent link="hand"/>
     <child link="finger_1"/>
     <origin xyz="0.03 0 0.04"/>
     <limit effort="100" velocity="1.0" lower="0" upper="-0.03"/>
+    <mimic joint="hand_finger_2" multiplier="-1"/>
   </joint>
   <xacro:make_link name="finger_1"
@@ -212,14 +206,13 @@
     rpy="0 0 0"
     color="Black"
-    mass="0.25"
+    mass="0.01"
     ixx="1640625.000000" ixy="0.000262" ixz="416666.656250"
     iyy="1453125.500000" iyz="0.000365"
     izz="593749.937500"/>
-  <joint name="hand-finger_2" type="prismatic">
+  <joint name="hand_finger_2" type="prismatic">
     <parent link="hand"/>
     <child link="finger_2"/>
     <origin xyz="-0.03 0 0.04"/>
     <limit effort="100" velocity="1.0" lower="0" upper="0.03"/>
-    <mimic joint="hand-finger" multiplier="-1"/>
   </joint>
   <xacro:make_link name="finger_2"
@@ -228,5 +221,5 @@
     rpy="0 0 3.14"
     color="Black"
-    mass="0.25"
+    mass="0.01"
     ixx="1640625.000000" ixy="0.000262" ixz="416666.656250"
     iyy="1453125.500000" iyz="0.000365"

Commit message: Debug failure of gripper planning

File: robot_modeling_ws/src/robot_description_pkg/urdf/mesh_arm.urdf (robot description, URDF)
Before this commit: robot penguin, 11 links, 10 joints
Joints:
- joint hand_finger_1: limit lower=0 upper=-0.03 effort=100 velocity=1.0 -> lower=-0.03 upper=0 effort=100 velocity=1.0

File: robot_modeling_ws/src/robot_description_pkg/urdf/mesh_arm.xacro (robot description, xacro)
@@ -198,5 +198,5 @@
     <child link="finger_1"/>
     <origin xyz="0.03 0 0.04"/>
-    <limit effort="100" velocity="1.0" lower="0" upper="-0.03"/>
+    <limit effort="100" velocity="1.0" lower="-0.03" upper="0"/>
     <mimic joint="hand_finger_2" multiplier="-1"/>
   </joint>
